File: LogicGate/LogicGate.kicad_pcb (KiCad board)
At the start: 2 copper layers, 78.7 x 71.1 mm, 16 parts, among them J1 Screw_Terminal_01x02, J2 Screw_Terminal_01x02, J3 Screw_Terminal_01x07, U1 IR2184, U2 IR2184

Commit message: latest route pcb
Parts:
- C1, C2, C3, C4, C5: value C_Polarized_US -> C; footprint TerminalBlock_Phoenix:TerminalBlock_Phoenix_MPT-0,5-2-2.54_1x02_P2.54mm_Horizontal -> Capacitor_THT:C_Disc_D7.5mm_W2.5mm_P5.00mm
- D1, D2: footprint TerminalBlock_Phoenix:TerminalBlock_Phoenix_MPT-0,5-2-2.54_1x02_P2.54mm_Horizontal -> Package_TO_SOT_THT:TO-220-2_Vertical
- R1, R2, R3, R4: footprint TerminalBlock_Phoenix:TerminalBlock_Phoenix_MPT-0,5-2-2.54_1x02_P2.54mm_Horizontal -> Resistor_THT:R_Axial_DIN0207_L6.3mm_D2.5mm_P7.62mm_Horizontal
- moved R2 51.2 mm to (171.4, 104.1), turned to 180 degrees
- moved R4 47.0 mm to (171.4, 116.8), turned to 180 degrees
- moved C5 44.0 mm to (179.7, 92.7), turned to 90 degrees
- moved D1 41.8 mm to (143.5, 78.4)
- moved R3 40.9 mm to (171.4, 111.8), turned to 180 degrees
- moved J2 29.2 mm to (111.5, 123.2)
- moved C3 28.8 mm to (141.0, 85.1)
- moved U1 28.4 mm to (143.5, 97.8)
- moved U2 28.4 mm to (143.5, 128.3)
- moved R1 28.2 mm to (171.4, 99.1), turned to 180 degrees
- moved C1 26.9 mm to (151.2, 85.1)
- moved C2 24.5 mm to (151.2, 114.3)
- moved D2 24.2 mm to (142.2, 108.9)
- moved J1 21.6 mm to (111.8, 92.7)
- moved J3 13.2 mm to (179.6, 119.7)
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Connections:
- C5 pad 1: VDD -> VCC
- J3 pad 7: VDD -> VCC
Routing:
- net VCC: track 0.00 -> 101.6 mm, vias 0 -> 2
- net Net-(J2-Pad1): track 0.00 -> 37.5 mm
- net Net-(J1-Pad1): track 0.00 -> 37.2 mm
- net Net-(J2-Pad2): track 0.00 -> 32.1 mm
- net Net-(J1-Pad2): track 0.00 -> 31.8 mm
- net Net-(R3-Pad2): track 0.00 -> 28.8 mm
- net Net-(R1-Pad2): track 0.00 -> 24.4 mm
- net Net-(R2-Pad2): track 0.00 -> 21.9 mm
- net Net-(R4-Pad2): track 0.00 -> 21.9 mm
- net Net-(C4-Pad1): track 0.00 -> 15.0 mm
- net Net-(C3-Pad1): track 0.00 -> 13.8 mm
- net Net-(J3-Pad6): track 0.00 -> 10.2 mm
- net Net-(J3-Pad3): track 0.00 -> 9.90 mm
- net Net-(J3-Pad4): track 0.00 -> 9.24 mm
- net Net-(J3-Pad5): track 0.00 -> 8.84 mm
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- added copper zone on B.Cu, net GND
- added copper zone on F.Cu, net GND
Other:
- board size 78.7 x 71.1 mm -> 79.4 x 71.1 mm
- board text added: "INPUT_1"
- board text added: "INPUT_2"
