File: LogicGate/LogicGate.kicad_sch (KiCad schematic)
At the start: 16 parts, among them J1 Screw_Terminal_01x02, J2 Screw_Terminal_01x02, J3 Screw_Terminal_01x07, U1 IR2184, U2 IR2184

Commit message: update LogicGate project
Parts:
- J3: footprint TerminalBlock_Phoenix:TerminalBlock_Phoenix_PT-1,5-6-3.5-H_1x06_P3.50mm_Horizontal -> TerminalBlock_Phoenix:TerminalBlock_Phoenix_PT-1,5-7-3.5-H_1x07_P3.50mm_Horizontal
Changed lines of the file:
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@@
       (effects (font (size 1.27 1.27)) hide)
     )
-    (property "Footprint" "TerminalBlock_Phoenix:TerminalBlock_Phoenix_PT-1,5-6-3.5-H_1x06_P3.50mm_Horizontal" (id 2) (at 187.96 78.74 0)
+    (property "Footprint" "TerminalBlock_Phoenix:TerminalBlock_Phoenix_PT-1,5-7-3.5-H_1x07_P3.50mm_Horizontal" (id 2) (at 187.96 78.74 0)
       (effects (font (size 1.27 1.27)) hide)
     )
@@
     )
     (path "/2fb78107-f191-46e4-b26d-54a2f7ca615a"
-      (reference "J3") (unit 1) (value "Screw_Terminal_01x07") (footprint "TerminalBlock_Phoenix:TerminalBlock_Phoenix_PT-1,5-6-3.5-H_1x06_P3.50mm_Horizontal")
+      (reference "J3") (unit 1) (value "Screw_Terminal_01x07") (footprint "TerminalBlock_Phoenix:TerminalBlock_Phoenix_PT-1,5-7-3.5-H_1x07_P3.50mm_Horizontal")
     )
     (path "/40c3bae4-5b67-4585-88ff-668d6966e76a"

Commit message: latest route pcb
Parts:
- C1, C2, C3, C4, C5: value C_Polarized_US -> C; footprint TerminalBlock_Phoenix:TerminalBlock_Phoenix_MPT-0,5-2-2.54_1x02_P2.54mm_Horizontal -> Capacitor_THT:C_Disc_D7.5mm_W2.5mm_P5.00mm; symbol Device:C_Polarized_US -> Device:C
- D1, D2: footprint TerminalBlock_Phoenix:TerminalBlock_Phoenix_MPT-0,5-2-2.54_1x02_P2.54mm_Horizontal -> Package_TO_SOT_THT:TO-220-2_Vertical
- R1, R2, R3, R4: footprint TerminalBlock_Phoenix:TerminalBlock_Phoenix_MPT-0,5-2-2.54_1x02_P2.54mm_Horizontal -> Resistor_THT:R_Axial_DIN0207_L6.3mm_D2.5mm_P7.62mm_Horizontal
Connections:
- net VDD is gone; now on net VCC: C5.1, J3.7 (Pin_7)
