File: PrimaryCore/PrimaryCore.kicad_sch (KiCad schematic)
At the start: 11 parts, among them J1 Screw_Terminal_01x02, J2 Screw_Terminal_01x06, J3 Screw_Terminal_01x02, Q1 Q_NMOS_DGS, Q2 Q_NMOS_DGS, Q3 Q_NMOS_DGS, Q4 Q_NMOS_DGS

Commit message: Change Cap footpackage p 10mm
Parts:
- C2: footprint Capacitor_THT:C_Disc_D7.5mm_W4.4mm_P5.00mm -> Capacitor_THT:C_Disc_D7.5mm_W5.0mm_P10.00mm
- C3: footprint Capacitor_THT:C_Disc_D3.8mm_W2.6mm_P2.50mm -> Capacitor_THT:C_Disc_D7.5mm_W5.0mm_P10.00mm
Changed lines of the file:
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@@
     (property "Reference" "C3" (id 0) (at 161.29 71.12 90))
     (property "Value" "270pF" (id 1) (at 161.29 73.66 90))
-    (property "Footprint" "Capacitor_THT:C_Disc_D3.8mm_W2.6mm_P2.50mm" (id 2) (at 165.1 77.7748 0)
+    (property "Footprint" "Capacitor_THT:C_Disc_D7.5mm_W5.0mm_P10.00mm" (id 2) (at 165.1 77.7748 0)
       (effects (font (size 1.27 1.27)) hide)
     )
@@
       (effects (font (size 1.27 1.27)) (justify left))
     )
-    (property "Footprint" "Capacitor_THT:C_Disc_D7.5mm_W4.4mm_P5.00mm" (id 2) (at 153.3652 87.63 0)
+    (property "Footprint" "Capacitor_THT:C_Disc_D7.5mm_W5.0mm_P10.00mm" (id 2) (at 153.3652 87.63 0)
       (effects (font (size 1.27 1.27)) hide)
     )
@@
     )
     (path "/b5058b0b-4178-433e-94f8-d98c100b0aed"
-      (reference "C2") (unit 1) (value "330pF") (footprint "Capacitor_THT:C_Disc_D7.5mm_W4.4mm_P5.00mm")
+      (reference "C2") (unit 1) (value "330pF") (footprint "Capacitor_THT:C_Disc_D7.5mm_W5.0mm_P10.00mm")
     )
     (path "/2b4a485a-9a24-4929-bea2-a453e8cb0507"
-      (reference "C3") (unit 1) (value "270pF") (footprint "Capacitor_THT:C_Disc_D3.8mm_W2.6mm_P2.50mm")
+      (reference "C3") (unit 1) (value "270pF") (footprint "Capacitor_THT:C_Disc_D7.5mm_W5.0mm_P10.00mm")
     )
     (path "/3a199f99-6e87-4483-bd70-76bbe63aedf3"

Commit message: latest route pcb
Parts:
- C1: footprint TerminalBlock_Phoenix:TerminalBlock_Phoenix_MPT-0,5-2-2.54_1x02_P2.54mm_Horizontal -> Capacitor_THT:CP_Radial_D18.0mm_P7.50mm
Changed lines of the file:
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@@
       (effects (font (size 1.27 1.27)) (justify left) hide)
     )
-    (property "Footprint" "TerminalBlock_Phoenix:TerminalBlock_Phoenix_MPT-0,5-2-2.54_1x02_P2.54mm_Horizontal" (id 2) (at 88.5952 88.9 0)
+    (property "Footprint" "Capacitor_THT:CP_Radial_D18.0mm_P7.50mm" (id 2) (at 88.5952 88.9 0)
       (effects (font (size 1.27 1.27)) hide)
     )
@@
     )
     (path "/e8fec1cf-a7c5-4355-bd03-2be882de8537"
-      (reference "C1") (unit 1) (value "C") (footprint "TerminalBlock_Phoenix:TerminalBlock_Phoenix_MPT-0,5-2-2.54_1x02_P2.54mm_Horizontal")
+      (reference "C1") (unit 1) (value "C") (footprint "Capacitor_THT:CP_Radial_D18.0mm_P7.50mm")
     )
     (path "/b5058b0b-4178-433e-94f8-d98c100b0aed"
