File: SecondaryCore/SecondaryCore.kicad_sch (KiCad schematic)
At the start: 7 parts, among them J1 Screw_Terminal_01x02, J2 Screw_Terminal_01x02

Commit message: Change Cap footpackage p 10mm
Parts:
- C1: footprint Capacitor_THT:C_Disc_D3.8mm_W2.6mm_P2.50mm -> Capacitor_THT:C_Disc_D7.5mm_W5.0mm_P10.00mm
- C2: footprint Capacitor_THT:C_Disc_D7.5mm_W4.4mm_P5.00mm -> Capacitor_THT:C_Disc_D7.5mm_W5.0mm_P10.00mm
Changed lines of the file:
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@@
       (effects (font (size 1.27 1.27)) (justify left))
     )
-    (property "Footprint" "Capacitor_THT:C_Disc_D7.5mm_W4.4mm_P5.00mm" (id 2) (at 112.7252 91.44 0)
+    (property "Footprint" "Capacitor_THT:C_Disc_D7.5mm_W5.0mm_P10.00mm" (id 2) (at 112.7252 91.44 0)
       (effects (font (size 1.27 1.27)) hide)
     )
@@
     (property "Reference" "C1" (id 0) (at 105.41 74.93 90))
     (property "Value" "270pF" (id 1) (at 105.41 77.47 90))
-    (property "Footprint" "Capacitor_THT:C_Disc_D3.8mm_W2.6mm_P2.50mm" (id 2) (at 109.22 81.5848 0)
+    (property "Footprint" "Capacitor_THT:C_Disc_D7.5mm_W5.0mm_P10.00mm" (id 2) (at 109.22 81.5848 0)
       (effects (font (size 1.27 1.27)) hide)
     )
@@
   (symbol_instances
     (path "/6ee110f7-4e65-4eb2-825f-8c02ae0dc741"
-      (reference "C1") (unit 1) (value "270pF") (footprint "Capacitor_THT:C_Disc_D3.8mm_W2.6mm_P2.50mm")
+      (reference "C1") (unit 1) (value "270pF") (footprint "Capacitor_THT:C_Disc_D7.5mm_W5.0mm_P10.00mm")
     )
     (path "/46176748-6355-4a13-9b3b-d86430f27056"
-      (reference "C2") (unit 1) (value "330pF") (footprint "Capacitor_THT:C_Disc_D7.5mm_W4.4mm_P5.00mm")
+      (reference "C2") (unit 1) (value "330pF") (footprint "Capacitor_THT:C_Disc_D7.5mm_W5.0mm_P10.00mm")
     )
     (path "/1e24d69a-d480-4335-a9f2-da0793ca1178"

Commit message: latest route pcb
Parts:
- C3: footprint TerminalBlock_Phoenix:TerminalBlock_Phoenix_MPT-0,5-2-2.54_1x02_P2.54mm_Horizontal -> Capacitor_THT:CP_Radial_D18.0mm_P7.50mm
Connections:
- net at D1.1 (+), J2.1 (Pin_1): now also C3.2; no longer C3.1
- net at D1.3 (-), J2.2 (Pin_2): now also C3.1; no longer C3.2
Other:
- moved on the sheet: C3
Changed lines of the file:
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@@
     (pin "2")
   )
-  (symbol (lib_id "Device:C") (at 152.4 81.28 0) (unit 1)
+  (symbol (lib_id "Device:C") (at 152.4 81.28 180) (unit 1)
     (in_bom yes) (on_board yes) (fields_autoplaced)
     (property "Reference" "C3" (id 0) (at 156.21 80.0099 0)
-      (effects (font (size 1.27 1.27)) (justify left))
+      (effects (font (size 1.27 1.27)) (justify right))
     )
     (property "Value" "C" (id 1) (at 156.21 82.5499 0)
-      (effects (font (size 1.27 1.27)) (justify left))
+      (effects (font (size 1.27 1.27)) (justify right))
     )
-    (property "Footprint" "TerminalBlock_Phoenix:TerminalBlock_Phoenix_MPT-0,5-2-2.54_1x02_P2.54mm_Horizontal" (id 2) (at 153.3652 85.09 0)
+    (property "Footprint" "Capacitor_THT:CP_Radial_D18.0mm_P7.50mm" (id 2) (at 151.4348 77.47 0)
       (effects (font (size 1.27 1.27)) hide)
     )
@@
     )
     (path "/1e24d69a-d480-4335-a9f2-da0793ca1178"
-      (reference "C3") (unit 1) (value "C") (footprint "TerminalBlock_Phoenix:TerminalBlock_Phoenix_MPT-0,5-2-2.54_1x02_P2.54mm_Horizontal")
+      (reference "C3") (unit 1) (value "C") (footprint "Capacitor_THT:CP_Radial_D18.0mm_P7.50mm")
     )
     (path "/a1b319a1-a99e-42d2-85f7-9644be3fa585"
